Commit message: Brought in velodyne description from repo and generated accessories.urdf

File: jackal_description/urdf/accessories.urdf.xacro (robot description, xacro)
@@ -10,16 +10,16 @@
   -->
   <!-- Macros to generate standoffs for offset payload mounting. -->
-  <xacro:include filename="$(find jackal_description)/urdf/accessories/standoffs.urdf.xacro" />
+  <xacro:include filename="accessories/standoffs.urdf.xacro" />
   <!-- This optional plate mounts both the upgraded GPS and the Velodyne 3D LIDAR. -->
-  <xacro:include filename="$(find jackal_description)/urdf/accessories/bridge_plate.urdf.xacro" />
+  <xacro:include filename="accessories/bridge_plate.urdf.xacro" />
   <!-- 2D Lidars -->
-  <xacro:include filename="$(find sick_tim)/urdf/sick_tim.urdf.xacro" />
-  <xacro:include filename="$(find lms1xx)/urdf/sick_lms1xx.urdf.xacro" />
-  <xacro:include filename="$(find jackal_description)/urdf/accessories/sick_lms1xx_inverted_mount.urdf.xacro" />
-  <xacro:include filename="$(find jackal_description)/urdf/accessories/sick_lms1xx_upright_mount.urdf.xacro" />
-  <xacro:include filename="$(find jackal_description)/urdf/accessories/hokuyo_utm30.urdf.xacro" />
-  <xacro:include filename="$(find jackal_description)/urdf/accessories/hokuyo_ust10.urdf.xacro" />
-  <xacro:include filename="$(find jackal_description)/urdf/accessories/vlp16_mount.urdf.xacro" />
-  <xacro:include filename="$(find jackal_description)/urdf/accessories/hdl32_mount.urdf.xacro" />
+  <!-- <xacro:include filename="$(find sick_tim)/urdf/sick_tim.urdf.xacro" /> -->
+  <!-- <xacro:include filename="$(find lms1xx)/urdf/sick_lms1xx.urdf.xacro" /> -->
+  <!-- <xacro:include filename="accessories/sick_lms1xx_inverted_mount.urdf.xacro" /> -->
+  <!-- <xacro:include filename="accessories/sick_lms1xx_upright_mount.urdf.xacro" /> -->
+  <!-- <xacro:include filename="accessories/hokuyo_utm30.urdf.xacro" /> -->
+  <!-- <xacro:include filename="accessories/hokuyo_ust10.urdf.xacro" /> -->
+  <xacro:include filename="accessories/vlp16_mount.urdf.xacro" />
+  <!-- <xacro:include filename="accessories/hdl32_mount.urdf.xacro" /> -->
   <!--
     Add Microstrain IMU. By default the Jackal comes equipped with an IMU linked to "imu_link". These extra
@@ -195,6 +195,6 @@
     - smart7              :: Novatel Smart7
   -->
-  <xacro:include filename="$(find jackal_description)/urdf/accessories/novatel_smart6.urdf.xacro" />
-  <xacro:include filename="$(find jackal_description)/urdf/accessories/novatel_smart7.urdf.xacro" />
+  <xacro:include filename="accessories/novatel_smart6.urdf.xacro" />
+  <xacro:include filename="accessories/novatel_smart7.urdf.xacro" />
   <xacro:if value="$(optenv JACKAL_NAVSAT 0)">
     <xacro:property name="mount" value="$(optenv JACKAL_NAVSAT_MOUNT rear)" />
@@ -257,6 +257,6 @@
   -->
   <!-- Common camera mounts and accessory URDFs. -->
-  <xacro:include filename="$(find jackal_description)/urdf/accessories/camera_mount.urdf.xacro" />
-  <xacro:include filename="$(find pointgrey_camera_description)/urdf/pointgrey_flea3.urdf.xacro" />
+  <!-- <xacro:include filename="accessories/camera_mount.urdf.xacro" /> -->
+  <!-- <xacro:include filename="$(find pointgrey_camera_description)/urdf/pointgrey_flea3.urdf.xacro" /> -->
   <!-- If enabled, generate the flea3 camera payload with a tilt of 30 degrees. -->
   <xacro:if value="$(optenv JACKAL_FLEA3 0)">
@@ -302,5 +302,5 @@
     </xacro:unless>
   </xacro:if>
-  <xacro:include filename="$(find jackal_description)/urdf/accessories/stereo_camera_mount.urdf.xacro" />
+  <xacro:include filename="accessories/stereo_camera_mount.urdf.xacro" />
   <!-- If enabled, generates a pair of flea3 cameras for stereo vision with a tilt of 30 degrees. -->
   <!-- Disabled temporarily due to metapackage issue. -->
@@ -338,5 +338,5 @@
   </xacro:if>
   <!-- If enabled, generate the bumblebee2 camera payload with a tilt of 0 degrees. -->
-  <xacro:include filename="$(find pointgrey_camera_description)/urdf/pointgrey_bumblebee2.urdf.xacro" />
+  <!-- <xacro:include filename="$(find pointgrey_camera_description)/urdf/pointgrey_bumblebee2.urdf.xacro" /> -->
   <!-- If enabled, generate the bumblebee2 camera payload with a tilt of 0 degrees. -->
   <!-- Disabled temporarily due to metapackage issue. -->
@@ -381,5 +381,5 @@
   </xacro:if>
   <!-- BlackflyS Camera -->
-  <xacro:include filename="$(find flir_camera_description)/urdf/flir_blackflys.urdf.xacro"/>
+  <!-- <xacro:include filename="$(find flir_camera_description)/urdf/flir_blackflys.urdf.xacro"/> -->
   <xacro:if value="$(optenv JACKAL_BLACKFLY 0)">
     <xacro:property name="prefix" value="$(optenv JACKAL_BLACKFLY_PREFIX front_camera)"/>
@@ -396,5 +396,5 @@
   <!-- Fender Accessories -->
   <xacro:if value="$(optenv JACKAL_FRONT_ACCESSORY_FENDER 0)">
-    <xacro:include filename="$(find jackal_description)/urdf/accessories/hokuyo_ust10.urdf.xacro" />
+    <xacro:include filename="accessories/hokuyo_ust10.urdf.xacro" />
     <xacro:if value="$(optenv JACKAL_FRONT_FENDER_UST10 0)">
       <xacro:hokuyo_ust10_mount

File: jackal_description/urdf/accessories/vlp16_mount.urdf.xacro (robot description, xacro)
@@ -1,4 +1,4 @@
 <robot xmlns:xacro="http://wiki.ros.org/xacro">
-  <xacro:include filename="$(find velodyne_description)/urdf/VLP-16.urdf.xacro" />
+  <xacro:include filename="../../../velodyne_description/urdf/VLP-16.urdf.xacro" />
   <xacro:macro name="vlp16_mount" params="prefix parent_link topic tower height:=0.1 *origin">
     <xacro:if value="${tower}">

File: jackal_description/urdf/jackal.urdf.xacro (robot description, xacro)
@@ -22,5 +22,5 @@
         <origin xyz="0 0 0" rpy="${PI/2} 0 0"/>
         <geometry>
-          <mesh filename="package://jackal_description/meshes/jackal-wheel.stl"/>
+          <mesh filename="../meshes/jackal-wheel.stl"/>
         </geometry>
         <material name="black" />
@@ -90,5 +90,5 @@
       <origin xyz="0 0 ${footprint_vertical_offset}" rpy="${PI/2} 0 ${PI/2}"/>
       <geometry>
-        <mesh filename="package://jackal_description/meshes/jackal-base.stl"/>
+        <mesh filename="../meshes/jackal-base.stl"/>
       </geometry>
       <material name="dark_grey" />
@@ -115,5 +115,5 @@
       <visual>
         <geometry>
-          <mesh filename="package://jackal_description/meshes/jackal-fender.stl"/>
+          <mesh filename="../meshes/jackal-fender.stl"/>
         </geometry>
         <material name="yellow" />
@@ -125,5 +125,5 @@
       <visual>
         <geometry>
-          <mesh filename="package://jackal_description/meshes/accessory_fender.stl"/>
+          <mesh filename="../meshes/accessory_fender.stl"/>
         </geometry>
         <material name="yellow" />
@@ -146,5 +146,5 @@
       <visual>
         <geometry>
-          <mesh filename="package://jackal_description/meshes/jackal-fender.stl"/>
+          <mesh filename="../meshes/jackal-fender.stl"/>
         </geometry>
         <material name="yellow" />
@@ -156,5 +156,5 @@
       <visual>
         <geometry>
-          <mesh filename="package://jackal_description/meshes/accessory_fender.stl"/>
+          <mesh filename="../meshes/accessory_fender.stl"/>
         </geometry>
         <material name="yellow" />
@@ -219,17 +219,17 @@
   </joint>
   <!-- Bring in simulation data for Gazebo. -->
-  <xacro:include filename="$(find jackal_description)/urdf/jackal.gazebo" />
+  <!-- <xacro:include filename="jackal.gazebo" /> -->
   <!-- Optional standard accessories, including their simulation data. The rendering
        of these into the final description is controlled by optenv variables, which
        default each one to off.-->
-  <xacro:include filename="$(find jackal_description)/urdf/accessories.urdf.xacro" />
+  <xacro:include filename="accessories.urdf.xacro" />
   <!-- OutdoorNav -->
   <xacro:arg name="outdoornav_enabled"       default="$(optenv OUTDOORNAV_ENABLED 0)" />
   <xacro:arg name="outdoornav_configuration" default="$(optenv OUTDOORNAV_CONFIGURATION standard)" />
-  <!-- OutdoorNav URDF Config -->
+  <!-- OutdoorNav URDF Config
   <xacro:if value="$(arg outdoornav_enabled)">
     <xacro:include filename="$(find cpr_onav_description)/urdf/outdoornav_description.urdf.xacro" />
     <xacro:outdoornav_sensors outdoornav_configuration="$(arg outdoornav_configuration)" />
-  </xacro:if>
+  </xacro:if> -->
   <!-- Optional custom includes. -->
   <xacro:include filename="$(optenv JACKAL_URDF_EXTRAS empty.urdf)" />
