Commit message: Set ENVVAR to include Velodyne lidar

File: jackal_description/urdf/accessories.urdf (robot description, URDF)
Before this commit: robot None, 0 links, 0 joints
Links:
- added link mid_vlp16_leg1; visual cylinder length=0.1 radius=0.003
- added link mid_vlp16_leg2; visual cylinder length=0.1 radius=0.003
- added link mid_vlp16_leg3; visual cylinder length=0.1 radius=0.003
- added link mid_vlp16_leg4; visual cylinder length=0.1 radius=0.003
- added link mid_vlp16_mount
- added link mid_vlp16_plate; visual box size=0.1 0.1 0.002
- added link velodyne, mass 0.1; visual mesh filename=package://velodyne_description/meshes/VLP16_scan.dae
- added link velodyne_base_link, mass 0.1; collision cylinder length=0.0717 radius=0.0516; visual mesh filename=package://velodyne_description/meshes/VLP16_base_1.dae
Joints:
- added joint mid_vlp16_leg1_joint: type fixed, parent mid_vlp16_mount, child mid_vlp16_leg1, origin xyz=0.05 0.05 0 rpy=0 0 0
- added joint mid_vlp16_leg2_joint: type fixed, parent mid_vlp16_mount, child mid_vlp16_leg2, origin xyz=0.05 -0.05 0 rpy=0 0 0
- added joint mid_vlp16_leg3_joint: type fixed, parent mid_vlp16_mount, child mid_vlp16_leg3, origin xyz=-0.05 0.05 0 rpy=0 0 0
- added joint mid_vlp16_leg4_joint: type fixed, parent mid_vlp16_mount, child mid_vlp16_leg4, origin xyz=-0.05 -0.05 0 rpy=0 0 0
- added joint mid_vlp16_mount_joint: type fixed, parent mid_mount, child mid_vlp16_mount, origin xyz=0 0 0 rpy=0 0 0
- added joint mid_vlp16_plate_joint: type fixed, parent mid_vlp16_mount, child mid_vlp16_plate, origin xyz=0 0 0.1 rpy=0 0 0
- added joint velodyne_base_mount_joint: type fixed, parent mid_vlp16_plate, child velodyne_base_link, origin xyz=0 0 0 rpy=0 0 0
- added joint velodyne_base_scan_joint: type fixed, parent velodyne_base_link, child velodyne, origin xyz=0 0 0.0377 rpy=0 0 0

File: jackal_description/urdf/accessories.urdf.xacro (robot description, xacro)
@@ -338,5 +338,4 @@
   </xacro:if>
   <!-- If enabled, generate the bumblebee2 camera payload with a tilt of 0 degrees. -->
-  <!-- <xacro:include filename="$(find pointgrey_camera_description)/urdf/pointgrey_bumblebee2.urdf.xacro" /> -->
   <!-- If enabled, generate the bumblebee2 camera payload with a tilt of 0 degrees. -->
   <!-- Disabled temporarily due to metapackage issue. -->
