Commit message: Working jackal_velodyne.xml with test_jackal_in_mujoco.py

File: jackal_description/urdf/jackal.urdf (robot description, URDF)
Before this commit: robot jackal, 21 links, 20 joints
Links:
- link velodyne: geometry visual mesh filename=../../velodyne_description/meshes/VLP16_scan.dae
- link velodyne_base_link: geometry collision cylinder length=0.0717 radius=0.0516; visual mesh filename=../../velodyne_description/meshes/VLP16_base_1.dae
